File: IV12-Clock/EDA/ME203_Project/ESP32Core.sch (KiCad schematic (older format))
At the start: 9 parts, among them J11 Conn_01x02, SW1 SW_Push, SW2 SW_Push, U4 ESP32-WROOM

Commit message: Code KWS, working on actual time.
Parts:
- removed J11: Conn_01x02, Connector_PinHeader_2.54mm:PinHeader_1x02_P2.54mm_Vertical, symbol Connector_Generic:Conn_01x02
- added J14: Conn_01x03, Connector_PinHeader_2.54mm:PinHeader_1x03_P2.54mm_Vertical, symbol Connector_Generic:Conn_01x03
- added J7: Micro_SD_Card, Connector_Card:microSD_HC_Wuerth_693072010801, symbol Connector:Micro_SD_Card
- added R20: 100kΩ, 0805, symbol SparkFun-Resistors:10KOHM-0603-1_10W-1%
Connections:
- net +3V3: now also J7.4 (VDD), R20.1
- net GND: now also J14.3 (Pin_3), J7.6 (VSS), J7.9 (SHIELD)
- net MISO-D19: now also J7.7 (DAT0)
- net MOSI-D18: now also J7.3 (CMD)
- net RXD0: now also J14.2 (Pin_2)
- net SCK-D5: now also J7.5 (CLK)
- net TXD0: now also J14.1 (Pin_1)
- net A10-D27 renamed SD-Select
- net SD-Select: now also J7.2 (DAT3/CD), R20.2
- net A11-D12 renamed A11-T5-D12
- net A5-D4 renamed A5-T0-D4
- net A6-D14 renamed A6-T6-D14
- net A7-D32 renamed A7-T9-D32
- net A9-D33 renamed A9-T8-D33
Other:
- moved on the sheet: C10, R18, R19, R24, R25, SW1, SW2, U4
