File: IV12-Clock/EDA/ME203_Project/MCU_RTC.sch (KiCad schematic (older format))
At the start: 3 parts

Commit message: Code KWS, working on actual time.
Parts:
- gave numbers to parts that had none: 1
Changed lines of the file:
@@
 $Descr A4 11693 8268
 encoding utf-8
-Sheet 3 7
+Sheet 3 8
 Title ""
 Date ""
@@
 	6550 3700 6950 3700
 $Comp
-L SparkFun-Batteries:BATTERY-20MM_SMD_4LEGS BT?
+L SparkFun-Batteries:BATTERY-20MM_SMD_4LEGS BT1
 U 1 1 5CB9110A
 P 6900 4000
-F 0 "BT?" V 6805 4178 45  0000 L CNN
+F 0 "BT1" V 6805 4178 45  0000 L CNN
 F 1 "BATTERY-20MM_SMD_4LEGS" V 6889 4178 45  0000 L CNN
 F 2 "BATTCON_20MM_4LEGS" H 6900 4250 20  0001 C CNN
