File: IV12-Clock/EDA/ME203_Project/MCU_TEMP.sch (KiCad schematic (older format))
At the start: 2 parts, among them U5 BMP280

Commit message: Code KWS, working on actual time.
Parts:
- added C12: 0.1µF, 0805, symbol SparkFun-Capacitors:1.0UF-0603-16V-10%
- C11: value 1.0µF -> 0.1µF
Connections:
- net +3V3: now also U5.2 (CSB), U5.5 (SDO), C12.1
- net GND: now also C12.2
- no-connect marks 2 -> 0
Other:
- note added: "One cap per power pin"
Changed lines of the file:
@@
 $Descr A4 11693 8268
 encoding utf-8
-Sheet 7 7
+Sheet 7 8
 Title ""
 Date ""
@@
 AR Path="/5CAA488B/5CCEF656" Ref="C?"  Part="1"
 AR Path="/5CCEB9C5/5CCEF656" Ref="C11"  Part="1"
+AR Path="/5CC63367/5CC72E77/5CCEF656" Ref="C?"  Part="1"
 F 0 "C11" H 5950 3850 45  0000 L CNN
-F 1 "1.0µF" H 5950 3750 45  0000 L CNN
+F 1 "0.1µF" H 5950 3750 45  0000 L CNN
 F 2 "0805" H 5850 3950 20  0001 C CNN
 F 3 "" H 5850 3700 50  0001 C CNN
@@
 U 1 1 5CCEF68F
 P 5200 3900
+AR Path="/5CCEB9C5/5CCEF68F" Ref="U5"  Part="1"
+AR Path="/5CC63367/5CC72E77/5CCEF68F" Ref="U?"  Part="1"
 F 0 "U5" H 5429 3996 50  0000 L CNN
 F 1 "BMP280" H 5429 3905 50  0000 L CNN
@@
 Wire Wire Line
 	5200 3500 5300 3500
-Connection ~ 5300 3500
 Wire Wire Line
 	5300 3500 5850 3500
@@
 AR Path="/5CCEFAB3" Ref="#PWR?"  Part="1"
 AR Path="/5CCEB9C5/5CCEFAB3" Ref="#PWR0125"  Part="1"
+AR Path="/5CC63367/5CC72E77/5CCEFAB3" Ref="#PWR?"  Part="1"
 F 0 "#PWR0125" H 5850 3250 50  0001 C CNN
 F 1 "+3.3V" H 5865 3573 50  0000 C CNN
@@
 AR Path="/5CCF2BFE" Ref="#GND?"  Part="1"
 AR Path="/5CCEB9C5/5CCF2BFE" Ref="#GND0125"  Part="1"
+AR Path="/5CC63367/5CC72E77/5CCF2BFE" Ref="#GND?"  Part="1"
 F 0 "#GND0125" H 5900 3750 45  0001 L BNN
 F 1 "GND" H 5850 3631 45  0000 C CNN
@@
 AR Path="/5CCF2CB5" Ref="#GND?"  Part="1"
 AR Path="/5CCEB9C5/5CCF2CB5" Ref="#GND0126"  Part="1"
+AR Path="/5CC63367/5CC72E77/5CCF2CB5" Ref="#GND?"  Part="1"
 F 0 "#GND0126" H 5350 4250 45  0001 L BNN
 F 1 "GND" H 5300 4131 45  0000 C CNN
@@
 Text HLabel 4550 3800 0    50   Input ~ 0
 SDA
-NoConn ~ 4800 3900
-NoConn ~ 4800 4000
 $Comp
 L SparkFun-PowerSymbols:GND #GND?
@@
 AR Path="/5CCF43BC" Ref="#GND?"  Part="1"
 AR Path="/5CCEB9C5/5CCF43BC" Ref="#GND0127"  Part="1"
+AR Path="/5CC63367/5CC72E77/5CCF43BC" Ref="#GND?"  Part="1"
 F 0 "#GND0127" H 4700 3950 45  0001 L BNN
 F 1 "GND" H 4650 3831 45  0000 C CNN
@@
 AR Path="/5CCF4A5F" Ref="#PWR?"  Part="1"
 AR Path="/5CCEB9C5/5CCF4A5F" Ref="#PWR0126"  Part="1"
+AR Path="/5CC63367/5CC72E77/5CCF4A5F" Ref="#PWR?"  Part="1"
 F 0 "#PWR0126" H 4650 3350 50  0001 C CNN
 F 1 "+3.3V" H 4665 3673 50  0000 C CNN
@@
 Wire Wire Line
 	4650 3600 4650 3500
+Wire Wire Line
+	4800 4000 4750 4000
+$Comp
+L power:+3.3V #PWR?
+U 1 1 5CD07D30
+P 4950 4400
+AR Path="/5CD07D30" Ref="#PWR?"  Part="1"
+AR Path="/5CCEB9C5/5CD07D30" Ref="#PWR0130"  Part="1"
+AR Path="/5CC63367/5CC72E77/5CD07D30" Ref="#PWR?"  Part="1"
+F 0 "#PWR0130" H 4950 4250 50  0001 C CNN
+F 1 "+3.3V" H 4965 4573 50  0000 C CNN
+F 2 "" H 4950 4400 50  0001 C CNN
+F 3 "" H 4950 4400 50  0001 C CNN
+	1    4950 4400
+	-1   0    0    -1
+$EndComp
+Wire Wire Line
+	4750 4550 4950 4550
+Wire Wire Line
+	4950 4550 4950 4400
+Wire Wire Line
+	4750 4000 4750 4550
+Connection ~ 5300 3500
+$Comp
+L SparkFun-Capacitors:1.0UF-0603-16V-10% C?
+U 1 1 5CD0870E
+P 6250 3700
+AR Path="/5CAA488B/5CD0870E" Ref="C?"  Part="1"
+AR Path="/5CCEB9C5/5CD0870E" Ref="C12"  Part="1"
+AR Path="/5CC63367/5CC72E77/5CD0870E" Ref="C?"  Part="1"
+F 0 "C12" H 6350 3850 45  0000 L CNN
+F 1 "0.1µF" H 6350 3750 45  0000 L CNN
+F 2 "0805" H 6250 3950 20  0001 C CNN
+F 3 "" H 6250 3700 50  0001 C CNN
+F 4 "CAP-00868" H 6358 3708 60  0001 L CNN "Field4"
+F 5 "0805" H 6450 3650 50  0000 C CNN "Size"
+	1    6250 3700
+	1    0    0    -1
+$EndComp
+$Comp
+L SparkFun-PowerSymbols:GND #GND?
+U 1 1 5CD08715
+P 6250 3800
+AR Path="/5CD08715" Ref="#GND?"  Part="1"
+AR Path="/5CCEB9C5/5CD08715" Ref="#GND0131"  Part="1"
+AR Path="/5CC63367/5CC72E77/5CD08715" Ref="#GND?"  Part="1"
+F 0 "#GND0131" H 6300 3750 45  0001 L BNN
+F 1 "GND" H 6250 3631 45  0000 C CNN
+F 2 "" H 6250 3700 60  0001 C CNN
+F 3 "" H 6250 3700 60  0001 C CNN
+	1    6250 3800
+	1    0    0    -1
+$EndComp
+Wire Wire Line
+	5850 3500 6250 3500
+Text Notes 5600 4100 0    50   ~ 0
+One cap per power pin
+Wire Wire Line
+	4800 3900 4750 3900
+Wire Wire Line
+	4750 3900 4750 4000
+Connection ~ 4750 4000
 $EndSCHEMATC
