File: IV12-Clock/EDA/ME203_Project/Main_Supply.sch (KiCad schematic (older format))
At the start: 8 parts, among them J4 Conn_01x02, J5 Conn_01x02, U3 TPS82140SILR

Commit message: Code KWS, working on actual time.
Parts:
- C7: footprint 1210 -> 1206; Size 1210 -> 1206
- R22, R23: footprint 0603 -> 0805; Size 0603 -> 0805
Changed lines of the file:
@@
 $Descr A4 11693 8268
 encoding utf-8
-Sheet 5 7
+Sheet 5 8
 Title ""
 Date ""
@@
 F 0 "C7" H 4608 3483 45  0000 L CNN
 F 1 "10µF" H 4608 3399 45  0000 L CNN
-F 2 "1210" H 4500 3550 20  0001 C CNN
+F 2 "1206" H 4500 3550 20  0001 C CNN
 F 3 "" H 4500 3300 50  0001 C CNN
 F 4 "CAP-09824" H 4608 3266 60  0001 L CNN "Field4"
-F 5 "1210" H 4608 3312 50  0000 L CNN "Size"
+F 5 "1206" H 4608 3312 50  0000 L CNN "Size"
 F 6 "50V" H 4608 3221 50  0000 L CNN "Potential"
 	1    4500 3300
@@
 F 0 "R22" V 6608 3268 45  0000 L CNN
 F 1 "300kΩ" V 6692 3268 45  0000 L CNN
-F 2 "0603" H 6650 3350 20  0001 C CNN
+F 2 "0805" H 6650 3350 20  0001 C CNN
 F 3 "" H 6650 3200 60  0001 C CNN
 F 4 "RES-10809" V 6734 3268 60  0001 L CNN "Field4"
-F 5 "0603" V 6650 3200 50  0001 C CNN "Size"
+F 5 "0805" V 6800 3350 50  0000 C CNN "Size"
 	1    6650 3200
 	0    1    1    0
@@
 F 0 "R23" V 6608 3668 45  0000 L CNN
 F 1 "100KΩ" V 6692 3668 45  0000 L CNN
-F 2 "0603" H 6650 3750 20  0001 C CNN
+F 2 "0805" H 6650 3750 20  0001 C CNN
 F 3 "" H 6650 3600 60  0001 C CNN
 F 4 "RES-07828" V 6734 3668 60  0001 L CNN "Field4"
-F 5 "0603" V 6650 3600 50  0001 C CNN "Size"
+F 5 "0805" V 6800 3650 50  0000 L CNN "Size"
 	1    6650 3600
 	0    1    1    0
