File: IV12-Clock/EDA/ME203_Project/Nixie_Interface.sch (KiCad schematic (older format))
At the start: 4 parts, among them J3 Conn_01x06, U2 CD40109

Commit message: Code KWS, working on actual time.
Parts:
- C4, C5: value 1.0µF -> 0.1µF
Changed lines of the file:
@@
 $Descr A4 11693 8268
 encoding utf-8
-Sheet 4 7
+Sheet 4 8
 Title ""
 Date ""
@@
 AR Path="/5CAB0187/5CAB68E1" Ref="C5"  Part="1"
 F 0 "C5" V 6500 2650 45  0000 L CNN
-F 1 "1.0µF" V 6400 2750 45  0000 R CNN
+F 1 "0.1µF" V 6400 2750 45  0000 R CNN
 F 2 "0805" V 6300 2650 45  0000 C CNN
 F 3 "" H 6250 2800 50  0001 C CNN
@@
 AR Path="/5CAB0187/5CAB68E9" Ref="C4"  Part="1"
 F 0 "C4" V 5200 3100 45  0000 R CNN
-F 1 "1.0µF" V 5100 3100 45  0000 R CNN
+F 1 "0.1µF" V 5100 3100 45  0000 R CNN
 F 2 "0805" V 5000 3000 45  0000 C CNN
 F 3 "" H 4950 2800 50  0001 C CNN
