File: IV12-Clock/EDA/ME203_Project/Nixie_PSU.sch (KiCad schematic (older format))
At the start: 16 parts, among them Q1 AO4294, T1 WE-FLEX_ER11_5, U1 LM3478SOIC8

Commit message: Code KWS, working on actual time.
Parts:
- CS1: value 380pF -> 360pF
- R1: value 1.2MΩ -> 2.2MΩ; Size (none) -> 0805
- R2: value 8.2KOHM-0603-1_10W-5% -> 12KΩ; footprint 0603 -> 0805; Size (none) -> 0805
- R3: value 300OHM-0603-1_10W-1% -> 3.3KΩ; footprint 0603 -> 0805; Size (none) -> 0805
Connections:
- net ~EN is gone; now on net GND: RF1.1
Changed lines of the file:
@@
 $Descr A4 11693 8268
 encoding utf-8
-Sheet 2 7
+Sheet 2 8
 Title ""
 Date ""
@@
 Wire Wire Line
 	4550 3950 4650 3950
-Text HLabel 4150 3950 0    50   Input ~ 0
-~EN
 $Comp
 L SparkFun-Capacitors:10UF-1210-50V-20% C1
@@
 P 8250 3550
 F 0 "R1" V 8208 3618 45  0000 L CNN
-F 1 "1.2MΩ" V 8292 3618 45  0000 L CNN
+F 1 "2.2MΩ" V 8292 3618 45  0000 L CNN
 F 2 "0603" H 8250 3700 20  0001 C CNN
 F 3 "" H 8250 3550 60  0001 C CNN
 F 4 "RES-10055" V 8292 3618 60  0001 L CNN "Field4"
+F 5 "0805" V 8400 3700 50  0000 C CNN "Size"
 	1    8250 3550
 	0    1    1    0
@@
 P 6150 3100
 F 0 "CS1" H 6258 3237 45  0000 L CNN
-F 1 "380pF" H 6258 3153 45  0000 L CNN
+F 1 "360pF" H 6258 3153 45  0000 L CNN
 F 2 "Capacitor_SMD:C_0603_1608Metric" H 6150 3350 20  0001 C CNN
 F 3 "" H 6150 3100 50  0001 C CNN
@@
 P 8250 4150
 F 0 "R2" V 8155 4218 45  0000 L CNN
-F 1 "8.2KOHM-0603-1_10W-5%" V 8239 4218 45  0000 L CNN
-F 2 "0603" H 8250 4300 20  0001 C CNN
+F 1 "12KΩ" V 8239 4218 45  0000 L CNN
+F 2 "0805" H 8250 4300 20  0001 C CNN
 F 3 "" H 8250 4150 60  0001 C CNN
-F 4 "RES-10646" V 8334 4218 60  0000 L CNN "Field4"
+F 4 "RES-10646" V 8334 4218 60  0001 L CNN "Field4"
+F 5 "0805" V 8350 4300 50  0000 C CNN "Size"
 	1    8250 4150
 	0    1    1    0
@@
 P 8250 4550
 F 0 "R3" V 8155 4618 45  0000 L CNN
-F 1 "300OHM-0603-1_10W-1%" V 8239 4618 45  0000 L CNN
-F 2 "0603" H 8250 4700 20  0001 C CNN
+F 1 "3.3KΩ" V 8239 4618 45  0000 L CNN
+F 2 "0805" H 8250 4700 20  0001 C CNN
 F 3 "" H 8250 4550 60  0001 C CNN
-F 4 "RES_10328" V 8334 4618 60  0000 L CNN "Field4"
+F 4 "RES_10328" V 8334 4618 60  0001 L CNN "Field4"
+F 5 "0805" V 8350 4700 50  0000 C CNN "Size"
 	1    8250 4550
 	0    1    1    0
@@
 Text HLabel 3650 3950 0    50   BiDi ~ 0
 GND
+$Comp
+L SparkFun-PowerSymbols:GND #GND09
+U 1 1 5CD81CFB
+P 4100 4000
+F 0 "#GND09" H 4150 3950 45  0001 L BNN
+F 1 "GND" H 4100 3831 45  0000 C CNN
+F 2 "" H 4100 3900 60  0001 C CNN
+F 3 "" H 4100 3900 60  0001 C CNN
+	1    4100 4000
+	1    0    0    -1
+$EndComp
+Wire Wire Line
+	4150 3950 4100 3950
+Wire Wire Line
+	4100 3950 4100 4000
 $EndSCHEMATC
