File: IV12-Clock/EDA/ME203_Project/DriverBoard/NixieDriver/NixieDriver.kicad_pcb (KiCad board)
At the start: 2 copper layers, 45.7 x 23.9 mm, 10 parts, among them J1 Conn_02x08_Counter_Clockwise, J2 Conn_01x06, J3 Conn_01x06, J4 Conn_02x08_Counter_Clockwise, U1 HV5530PG-G-44PQF

Commit message: Code KWS, working on actual time.
Parts:
- C1: value 0.1UF-0603-100V-10% -> 0.1UF-0805-100V; footprint 0603 -> 0805
