File: IV12-Clock/EDA/ME203_Project/DriverBoard/NixieDriver/NixieDriver.sch (KiCad schematic (older format))
At the start: 10 parts, among them J1 Conn_02x08_Counter_Clockwise, J2 Conn_01x06, J3 Conn_01x06, J4 Conn_02x08_Counter_Clockwise, U1 HV5530PG-G-44PQF

Commit message: Code KWS, working on actual time.
Parts:
- C1: value 0.1UF-0603-100V-10% -> 0.1UF-0805-100V; footprint 0603 -> 0805
Changed lines of the file:
@@
 AR Path="/5CAF5F4B" Ref="C1"  Part="1"
 F 0 "C1" H 6558 6150 45  0000 L CNN
-F 1 "0.1UF-0603-100V-10%" H 6558 6161 45  0001 L CNN
-F 2 "0603" H 6450 6350 20  0001 C CNN
+F 1 "0.1UF-0805-100V" H 6558 6161 45  0001 L CNN
+F 2 "0805" H 6450 6350 20  0001 C CNN
 F 3 "" H 6450 6100 50  0001 C CNN
 F 4 "CAP-08390" H 6558 6108 60  0001 L CNN "Field4"
